File: n40a8c/n40a8c.kicad_sch (KiCad schematic)
At the start: 111 parts, among them J1 Conn_01x02_Pin, J2 Conn_01x02_Pin, SW1 CPG151101S11-16, SW10 CPG151101S11-16, SW11 CPG151101S11-16, SW12 CPG151101S11-16, SW13 CPG151101S11-16, SW14 CPG151101S11-16, SW15 CPG151101S11-16, SW16 CPG151101S11-16, SW17 CPG151101S11-16, SW18 CPG151101S11-16, SW19 CPG151101S11-16, SW2 CPG151101S11-16, SW20 CPG151101S11-16, SW21 CPG151101S11-16, SW22 CPG151101S11-16, SW23 CPG151101S11-16, SW24 CPG151101S11-16, SW25 CPG151101S11-16, SW26 CPG151101S11-16, SW27 CPG151101S11-16, SW28 CPG151101S11-16, SW29 CPG151101S11-16, SW3 CPG151101S11-16, SW30 CPG151101S11-16, SW31 CPG151101S11-16, SW32 CPG151101S11-16, SW33 CPG151101S11-16, SW34 CPG151101S11-16, SW35 CPG151101S11-16, SW36 CPG151101S11-16, SW37 CPG151101S11-16, SW38 CPG151101S11-16, SW39 CPG151101S11-16, SW4 CPG151101S11-16, SW40 CPG151101S11-16, SW41 CPG151101S11-16, SW42 CPG151101S11-16, SW5 CPG151101S11-16, SW6 CPG151101S11-16, SW7 CPG151101S11-16, SW8 CPG151101S11-16, SW9 CPG151101S11-16, U1 XIAO-nRF52840-SMD

Commit message: M2→M2.6
Parts:
- H1, H2, H3, H4: footprint cscslib:MountingHole_M2_plating -> cscslib:MountingHole_M2.6_plating
Changed lines of the file:
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@@
 			)
 		)
-		(property "Footprint" "cscslib:MountingHole_M2_plating"
+		(property "Footprint" "cscslib:MountingHole_M2.6_plating"
 			(at 170.18 25.4 0)
 			(effects
@@
 			)
 		)
-		(property "Footprint" "cscslib:MountingHole_M2_plating"
+		(property "Footprint" "cscslib:MountingHole_M2.6_plating"
 			(at 170.18 35.56 0)
 			(effects
@@
 			)
 		)
-		(property "Footprint" "cscslib:MountingHole_M2_plating"
+		(property "Footprint" "cscslib:MountingHole_M2.6_plating"
 			(at 170.18 30.48 0)
 			(effects
@@
 			)
 		)
-		(property "Footprint" "cscslib:MountingHole_M2_plating"
+		(property "Footprint" "cscslib:MountingHole_M2.6_plating"
 			(at 170.18 40.64 0)
 			(effects

Commit message: M2.6→M3
Parts:
- H1, H2, H3, H4: footprint cscslib:MountingHole_M2.6_plating -> cscslib:MountingHole_M3_plating_truss
Changed lines of the file:
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@@
 			)
 		)
-		(property "Footprint" "cscslib:MountingHole_M2.6_plating"
+		(property "Footprint" "cscslib:MountingHole_M3_plating_truss"
 			(at 170.18 25.4 0)
 			(effects
@@
 			)
 		)
-		(property "Footprint" "cscslib:MountingHole_M2.6_plating"
+		(property "Footprint" "cscslib:MountingHole_M3_plating_truss"
 			(at 170.18 35.56 0)
 			(effects
@@
 			)
 		)
-		(property "Footprint" "cscslib:MountingHole_M2.6_plating"
+		(property "Footprint" "cscslib:MountingHole_M3_plating_truss"
 			(at 170.18 30.48 0)
 			(effects
@@
 			)
 		)
-		(property "Footprint" "cscslib:MountingHole_M2.6_plating"
+		(property "Footprint" "cscslib:MountingHole_M3_plating_truss"
 			(at 170.18 40.64 0)
 			(effects
