File: n40a8c/n40a8c_bottom.kicad_pcb (KiCad board)
At the start: 2 copper layers, 267.9 x 104.9 mm, 4 parts

Commit message: revise keysocket footprint. revise production pcb data.
Other:
- board text removed: "+"
- board text removed: "-"
Changed lines of the file:
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@@
-		)
-	)
-	(gr_text "-"
-		(at 175.617335 33.932841 0)
-		(layer "B.SilkS")
-		(effects
-			(font
-				(size 1 1)
-				(thickness 0.15)
-			)
-			(justify mirror)
-		)
-	)
-	(gr_text "+"
-		(at 182.761091 33.93284 0)
-		(layer "B.SilkS")
-		(effects
-			(font
-				(size 1 1)
-				(thickness 0.15)
-			)
-			(justify mirror)
-		)
-	)
-	(gr_text "+"
-		(at 186.332969 41.076598 0)
-		(layer "B.SilkS")
-		(effects
-			(font
-				(size 1 1)
-				(thickness 0.15)
-			)
-			(justify left bottom mirror)
 		)
 	)
@@
 		)
 	)
-	(gr_text "-"
-		(at 186.332969 35.718779 0)
-		(layer "B.SilkS")
-		(effects
-			(font
-				(size 1 1)
-				(thickness 0.15)
-			)
-			(justify left bottom mirror)
-		)
-	)
