File: n40a8c/n40a8c_pcb.kicad_pcb (KiCad board)
At the start: 2 copper layers, 267.9 x 104.9 mm, 107 parts, among them J1 Conn_01x02_Pin, J2 Conn_01x02_Pin, SW1 CPG151101S11-16, SW10 CPG151101S11-16, SW11 CPG151101S11-16, SW12 CPG151101S11-16, SW13 CPG151101S11-16, SW14 CPG151101S11-16, SW15 CPG151101S11-16, SW16 CPG151101S11-16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

Commit message: revise keysocket footprint. revise production pcb data.
Parts:
- moved SW_HPWR1 0.30 mm to (187.8, 25.6)
- moved SW_HPWR2 0.30 mm to (187.8, 25.6)
Other:
- outline, holes or cut-outs redrawn
