File: n42a7c/n42a7c_p.kicad_pcb (KiCad board)
At the start: 2 copper layers, 265.5 x 105.1 mm, 111 parts, among them J1 Conn_01x02, J2 Conn_01x03, SW1 CPG151101S11-16, SW10 CPG151101S11-16, SW11 CPG151101S11-16, SW12 CPG151101S11-16, SW13 CPG151101S11-16, SW14 CPG151101S11-16, SW15 CPG151101S11-16, SW16 CPG151101S11-16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

Commit message: create plate
Parts:
- removed H1, H2, H3, H4: MountingHole_Pad, cscslib:MountingHole_M3_plating_truss
Other:
- board size 265.5 x 105.1 mm -> 265.5 x 103.7 mm
