File: n42a7c/n42a7c_p.kicad_pcb (KiCad board)
At the start: 2 copper layers, 265.5 x 105.1 mm, 113 parts, among them J1 S2B-PH-SM4-TB, J2 S2B-PH-SM4-TB, J3 S2B-PH-SM4-TB, SW1 CPG151101S11-16, SW10 CPG151101S11-16, SW11 CPG151101S11-16, SW12 CPG151101S11-16, SW13 CPG151101S11-16, SW14 CPG151101S11-16, SW15 CPG151101S11-16, SW16 CPG151101S11-16, SW17 CPG151101S11-16, SW18 CPG151101S11-16, SW19 CPG151101S11-16, SW2 CPG151101S11-16, SW20 CPG151101S11-16, SW21 CPG151101S11-16, SW22 CPG151101S11-16, SW23 CPG151101S11-16, SW24 CPG151101S11-16, SW25 CPG151101S11-16, SW26 CPG151101S11-16, SW27 CPG151101S11-16, SW28 CPG151101S11-16, SW29 CPG151101S11-16, SW3 CPG151101S11-16, SW30 CPG151101S11-16, SW31 CPG151101S11-16, SW32 CPG151101S11-16, SW33 CPG151101S11-16, SW34 CPG151101S11-16, SW35 CPG151101S11-16, SW36 CPG151101S11-16, SW37 CPG151101S11-16, SW38 CPG151101S11-16, SW39 CPG151101S11-16, SW4 CPG151101S11-16, SW40 CPG151101S11-16, SW41 CPG151101S11-16, SW42 CPG151101S11-16, SW5 CPG151101S11-16, SW6 CPG151101S11-16, SW7 CPG151101S11-16, SW8 CPG151101S11-16, SW9 CPG151101S11-16, U1 XIAO-nRF52840-SMD

Commit message: create plate / production PCB
Parts:
- removed H1, H2, H3, H4: MountingHole_Pad, cscslib:MountingHole_M3_plating_truss
Other:
- board size 265.5 x 105.1 mm -> 265.5 x 103.7 mm

Commit message: create plate/production PCB
Parts:
- removed REF**: JST_PH_S2B-PH-K_1x02_P2.00mm_Horizontal, Connector_JST:JST_PH_S2B-PH-K_1x02_P2.00mm_Horizontal
- added J4: S2B-PH-SM4-TB, Connector_JST:JST_PH_S2B-PH-K_1x02_P2.00mm_Horizontal, B.Cu at (185.2, 37.6)
- moved SW35 2.38 mm to (30.4, 105.4)
- moved SW36 2.38 mm to (54.2, 105.4)
- moved D35 2.38 mm to (37.5, 107.8)
- moved D36 2.38 mm to (61.3, 107.8)
- moved D41 2.38 mm to (245.9, 107.8)
- moved SW41 2.38 mm to (238.7, 105.4)
- moved D42 2.38 mm to (269.7, 107.8)
- moved DI8 2.38 mm to (273.8, 107.8)
- moved DS8 2.38 mm to (273.8, 100.6)
- moved SW42 2.38 mm to (262.5, 105.4)
Routing:
- net IO 6: track 360.9 -> 363.3 mm
- net IO 7: track 354.0 -> 356.4 mm
- net Net-(D39-K): track 96.1 -> 98.5 mm
- net IO 4: track 355.0 -> 357.4 mm
- net IO 3: track 296.7 -> 299.1 mm
- net INTR: track 424.2 -> 424.8 mm
- net Net-(D35-K): track 119.7 -> 120.3 mm
- net IO 5: track 384.3 -> 383.7 mm
Other:
- outline, holes or cut-outs redrawn
- board text added: "Fn1"
- board text added: "Fn2"
- board text added: "POW"
- board text added: "n42a7c Rev 1.1 Jul. 2025 Designed by @_hatano_"
- board text removed: "n42a7c Rev 1.0 Jun. 2025 Designed by @_hatano_"

Commit message: revise
Parts:
- removed J1: S2B-PH-SM4-TB, Connector_JST:JST_PH_S2B-PH-SM4-TB_1x02-1MP_P2.00mm_Horizontal
- removed SW_DR1, SW_DR2: SKTDLDE010, cscslib:SKTDLDE010
- removed SW_HPWR1: SSSS811101, cscslib:SSSS811101
- added SW_D1: SKTDLDE010, cscslib:SKTDLDE010, B.Cu at (194.1, 23.8)
- added SW_D2: SKTDLDE010, cscslib:SKTDLDE010, B.Cu at (188.4, 23.8)
- added SW_PWR1: SSSS811101, cscslib:SSSS811101, B.Cu at (180.7, 24.4)
- J2, J3: value S2B-PH-SM4-TB -> ~
- J4: value S2B-PH-SM4-TB -> S2B-PH-K
- moved DI6 2.38 mm to (273.8, 88.7)
- moved DS6 2.38 mm to (273.8, 81.6)
- moved J4 0.60 mm to (185.8, 37.6)
Routing:
- net INTR: track 424.8 -> 428.4 mm
- net IO 5: track 383.7 -> 386.6 mm
- net Net-(D30-K): track 96.4 -> 98.8 mm
- net Net-(J1-Pin_1): track 30.1 -> 32.0 mm
- net IO 0: track 133.8 -> 133.0 mm
- net BAT-: track 45.4 -> 46.0 mm
Other:
- outline, holes or cut-outs redrawn
- board text removed: "Fn1"
- board text removed: "Fn2"
- board text removed: "POW"
