File: n42a7c/n42a7c_p.kicad_pcb (KiCad board)
At the start: 2 copper layers, 265.5 x 103.7 mm, 108 parts, among them J4 S2B-PH-K, SW1 CPG151101S11-16, SW10 CPG151101S11-16, SW11 CPG151101S11-16, SW12 CPG151101S11-16, SW13 CPG151101S11-16, SW14 CPG151101S11-16, SW15 CPG151101S11-16, SW16 CPG151101S11-16, SW17 CPG151101S11-16, SW18 CPG151101S11-16, SW19 CPG151101S11-16, SW2 CPG151101S11-16, SW20 CPG151101S11-16, SW21 CPG151101S11-16, SW22 CPG151101S11-16, SW23 CPG151101S11-16, SW24 CPG151101S11-16, SW25 CPG151101S11-16, SW26 CPG151101S11-16, SW27 CPG151101S11-16, SW28 CPG151101S11-16, SW29 CPG151101S11-16, SW3 CPG151101S11-16, SW30 CPG151101S11-16, SW31 CPG151101S11-16, SW32 CPG151101S11-16, SW33 CPG151101S11-16, SW34 CPG151101S11-16, SW35 CPG151101S11-16, SW36 CPG151101S11-16, SW37 CPG151101S11-16, SW38 CPG151101S11-16, SW39 CPG151101S11-16, SW4 CPG151101S11-16, SW40 CPG151101S11-16, SW41 CPG151101S11-16, SW42 CPG151101S11-16, SW5 CPG151101S11-16, SW6 CPG151101S11-16, SW7 CPG151101S11-16, SW8 CPG151101S11-16, SW9 CPG151101S11-16, U1 XIAO-nRF52840-SMD

Commit message: regen production pcb data
Routing:
- net Net-(D24-K): track 134.9 -> 131.9 mm
- net IO 4: track 357.4 -> 354.9 mm
- net Net-(J1-Pin_1): track 32.0 -> 30.1 mm
- net IO 3: track 299.1 -> 297.2 mm
- net IO 5: track 386.6 -> 385.0 mm
- net IO 2: track 224.7 -> 223.0 mm
- net BAT-: track 46.0 -> 45.0 mm
- net IO 0: track 133.0 -> 132.1 mm
- net INTR: track 428.4 -> 427.8 mm
Other:
- outline, holes or cut-outs redrawn
- board text added: "6.5mm spacer"
- board text added: "J1"
- board text added: "PHconn"
- board text added: "Socket"
