File: n42a7c/plate/n42a7c_b.kicad_pcb (KiCad board)
At the start: 2 copper layers, 265.5 x 105.1 mm, 4 parts

Commit message: create plate / production PCB
Other:
- outline, holes or cut-outs redrawn
- board text added: "7.0mm spacer"
- board text added: "CON"
- board text added: "M3x5 ramimate"
- board text added: "PHconn SMD"
- board text added: "PON"
- board text added: "POWER"
- board text added: "foot"

Commit message: create plate/production PCB
Other:
- outline, holes or cut-outs redrawn
- board text added: "n42a7c Rev 1.1 Jul. 2025 Designed by @_hatano_"
- board text removed: "n42a7c Rev 1.0 Jun. 2025 Designed by @_hatano_"

Commit message: create production plate
Other:
- outline, holes or cut-outs redrawn
Changed lines of the file:
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@@
 	)
 	(gr_circle
-		(center 175.914696 23.217168)
-		(end 175.61704 23.217168)
+		(center 269.081476 41.67191)
+		(end 273.081476 41.67191)
+		(stroke
+			(width 0.15)
+			(type solid)
+		)
+		(fill no)
+		(layer "B.Cu")
+	)
+	(gr_circle
+		(center 21.431232 111.323344)
+		(end 25.431232 111.323344)
+		(stroke
+			(width 0.15)
+			(type solid)
+		)
+		(fill no)
+		(layer "B.Cu")
+	)
+	(gr_circle
+		(center 271.462272 111.323344)
+		(end 275.462272 111.323344)
+		(stroke
+			(width 0.15)
+			(type solid)
+		)
+		(fill no)
+		(layer "B.Cu")
+	)
+	(gr_circle
+		(center 23.81252 41.67191)
+		(end 27.81252 41.67191)
+		(stroke
+			(width 0.15)
+			(type solid)
+		)
+		(fill no)
+		(layer "B.Cu")
+	)
+	(gr_circle
+		(center 176.807664 23.217168)
+		(end 176.510008 23.217168)
 		(stroke
 			(width 0.15)
@@
 	)
 	(gr_circle
-		(center 183.356096 36.611688)
-		(end 183.951408 36.611688)
-		(stroke
-			(width 0.1)
-			(type default)
-		)
-		(fill no)
-		(layer "Cmts.User")
-	)
-	(gr_circle
-		(center 185.210784 37.611688)
-		(end 185.737343 37.611688)
-		(stroke
-			(width 0.1)
-			(type solid)
-		)
-		(fill no)
-		(layer "Cmts.User")
-	)
-	(gr_circle
 		(center 153.590625 104.775)
 		(end 154.781252 104.775002)
@@
 		(layer "Eco2.User")
 	)
-	(gr_rect
-		(start 175.060784 32.011688)
-		(end 187.060784 41.211688)
-		(stroke
-			(width 0.15)
-			(type solid)
-		)
-		(fill no)
-		(locked yes)
-		(layer "Eco2.User")
-	)
-	(gr_circle
-		(center 269.081476 41.67191)
-		(end 273.081476 41.67191)
-		(stroke
-			(width 0.15)
-			(type solid)
-		)
-		(fill no)
-		(layer "Eco2.User")
-	)
-	(gr_line
-		(start 173.533448 44.053088)
-		(end 173.533449 22.621856)
-		(stroke
-			(width 0.15)
-			(type solid)
-		)
-		(layer "Eco2.User")
-	)
-	(gr_circle
-		(center 21.431232 111.323344)
-		(end 25.431232 111.323344)
-		(stroke
-			(width 0.15)
-			(type solid)
-		)
-		(fill no)
-		(layer "Eco2.User")
-	)
-	(gr_circle
-		(center 271.462272 111.323344)
-		(end 275.462272 111.323344)
-		(stroke
-			(width 0.15)
-			(type solid)
-		)
-		(fill no)
-		(layer "Eco2.User")
-	)
 	(gr_line
 		(start 237.827144 35.71872)
 		(end 230.088088 35.718779)
-		(stroke
-			(width 0.15)
-			(type solid)
-		)
-		(layer "Eco2.User")
-	)
-	(gr_line
-		(start 155.078776 22.621856)
-		(end 155.078776 44.053088)
-		(stroke
-			(width 0.15)
-			(type solid)
-		)
-		(layer "Eco2.User")
-	)
-	(gr_circle
-		(center 23.81252 41.67191)
-		(end 27.81252 41.67191)
-		(stroke
-			(width 0.15)
-			(type solid)
-		)
-		(fill no)
-		(layer "Eco2.User")
-	)
-	(gr_line
-		(start 155.078776 44.053088)
-		(end 173.533448 44.053088)
 		(stroke
 			(width 0.15)
@@
 	)
 	(gr_rect
-		(start 175.060784 33.161688)
-		(end 187.060784 40.061688)
-		(stroke
-			(width 0.15)
-			(type solid)
-		)
-		(fill no)
+		(start 175.656096 33.161688)
+		(end 187.656096 40.061688)
+		(stroke
+			(width 0.15)
+			(type solid)
+		)
+		(fill no)
+		(layer "Edge.Cuts")
+	)
+	(gr_line
+		(start 155.078776 22.621875)
+		(end 173.533449 22.621856)
+		(stroke
+			(width 0.15)
+			(type default)
+		)
 		(layer "Edge.Cuts")
 	)
@@
 			(width 0.15)
 			(type default)
-		)
-		(layer "Edge.Cuts")
-	)
-	(gr_line
-		(start 173.533448 22.621875)
-		(end 155.078776 22.621875)
-		(stroke
-			(width 0.15)
-			(type solid)
 		)
 		(layer "Edge.Cuts")
@@
 		)
 	)
-	(gr_text "7.0mm\nspacer"
-		(at 254 144.85 0)
-		(layer "Dwgs.User")
+	(gr_text "POWER"
+		(at 180.677192 23.514824 -0)
+		(layer "B.SilkS")
 		(effects
 			(font
@@
 				(thickness 0.15)
 			)
-		)
-	)
-	(gr_text "POWER"
-		(at 180.677192 23.514824 0)
-		(layer "Dwgs.User")
+			(justify mirror)
+		)
+	)
+	(gr_text "PON"
+		(at 194.071712 23.81248 -0)
+		(layer "B.SilkS" knockout)
 		(effects
 			(font
@@
 				(thickness 0.15)
 			)
-		)
-	)
-	(gr_text "foot"
-		(at 262.5 151.2 0)
-		(layer "Dwgs.User")
+			(justify mirror)
+		)
+	)
+	(gr_text "CON"
+		(at 188.416248 23.81248 -0)
+		(layer "B.SilkS" knockout)
 		(effects
 			(font
@@
 				(thickness 0.15)
 			)
-		)
-	)
-	(gr_text "PON"
-		(at 194.071712 23.81248 0)
-		(layer "Dwgs.User" knockout)
+			(justify mirror)
+		)
+	)
+	(gr_text "7.0mm\nspacer"
+		(at 254 144.85 0)
+		(layer "Dwgs.User")
 		(effects
 			(font
@@
 		)
 	)
-	(gr_text "M3x5 ramimate"
-		(at 253.95 137.75 0)
+	(gr_text "foot"
+		(at 262.5 151.2 0)
 		(layer "Dwgs.User")
 		(effects
@@
 		)
 	)
-	(gr_text "CON"
-		(at 188.416248 23.81248 0)
-		(layer "Dwgs.User" knockout)
+	(gr_text "M3x5 ramimate"
+		(at 253.95 137.75 0)
+		(layer "Dwgs.User")
 		(effects
 			(font

Commit message: regen production pcb data
Other:
- board text added: "6.5mm spacer"
- board text added: "PHconn"
- board text added: "Socket"
